File: _autosave-lm224-3lows-1hi.kicad_pcb (KiCad board)
At the start: 2 copper layers, 144.6 x 105.9 mm, 38 parts, among them J1 Power, J2 To LEDs, Q1 IRLB8721, Q2 IRLB8721, Q3 IRF5210L, Q4 IRLB8721, Q5 IRLB8721, U1 LM224

Commit message: Ok more stuff
Parts:
- RV1: value 10k -> To 10k Pot - Master Brightness
- RV2: value 10k -> To 10k Pot - Red
- RV3: value 10k -> To 10k Pot - Blue
- RV4: value 10k -> To 10k Pot - Green
Other:
- board text added: "+12VDC"
- board text added: "12VDC"
- board text added: "12VDC out"
- board text added: "GND"
- board text added: "GND Blue"
- board text added: "GND Green"
- board text added: "GND Red"
Changed lines of the file:
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@@
     (property "Sheetname" "")
     (attr through_hole)
-    (fp_text reference "J1" (at 2.54 -6.26 90) (layer "F.SilkS")
-      (effects (font (size 1 1) (thickness 0.15)))
-    )
-    (fp_text value "Power" (at 2.54 5.66 90) (layer "F.Fab")
+    (fp_text reference "J1" (at 2.6212 -7.163) (layer "F.SilkS")
+      (effects (font (size 1 1) (thickness 0.15)))
+    )
+    (fp_text value "Power" (at 9.022 -0.559) (layer "F.Fab")
       (effects (font (size 1 1) (thickness 0.15)))
     )
@@
       (effects (font (size 1 1) (thickness 0.15)))
     )
-    (fp_text value "10k" (at 5.08 5.66) (layer "F.Fab")
+    (fp_text value "To 10k Pot - Red" (at 4.8818 6.1466) (layer "F.SilkS")
       (effects (font (size 1 1) (thickness 0.15)))
     )
@@
       (effects (font (size 1 1) (thickness 0.15)))
     )
-    (fp_text value "10k" (at 5.08 5.66) (layer "F.Fab")
+    (fp_text value "To 10k Pot - Master Brightness" (at 5.1308 6.2992) (layer "F.SilkS")
       (effects (font (size 1 1) (thickness 0.15)))
     )
@@
     (property "Sheetname" "")
     (attr through_hole)
-    (fp_text reference "J2" (at 7.62 -6.26 90) (layer "F.SilkS")
-      (effects (font (size 1 1) (thickness 0.15)))
-    )
-    (fp_text value "To LEDs" (at 7.62 5.66 90) (layer "F.Fab")
+    (fp_text reference "J2" (at 19.7612 -0.2796 180) (layer "F.SilkS")
+      (effects (font (size 1 1) (thickness 0.15)))
+    )
+    (fp_text value "To LEDs" (at -4.4704 -0.0764 180) (layer "F.Fab")
       (effects (font (size 1 1) (thickness 0.15)))
     )
@@
       (effects (font (size 1 1) (thickness 0.15)))
     )
-    (fp_text value "10k" (at 5.08 5.66) (layer "F.Fab")
+    (fp_text value "To 10k Pot - Blue" (at 5.1358 6.1974) (layer "F.SilkS")
       (effects (font (size 1 1) (thickness 0.15)))
     )
@@
     (property "Sheetname" "")
     (attr through_hole)
-    (fp_text reference "U1" (at 3.81 -2.33 90) (layer "F.SilkS")
+    (fp_text reference "U1" (at 10.8612 7.5488 180) (layer "F.SilkS")
       (effects (font (size 1 1) (thickness 0.15)))
     )
@@
       (effects (font (size 1 1) (thickness 0.15)))
     )
-    (fp_text value "10k" (at 5.08 5.66) (layer "F.Fab")
+    (fp_text value "To 10k Pot - Green" (at 5.08 6.2482) (layer "F.SilkS")
       (effects (font (size 1 1) (thickness 0.15)))
     )
@@
   )
   (gr_rect (start 297.1292 0) (end 152.5016 105.8672) (layer "Edge.Cuts") (width 0.1) (fill none))
+  (gr_text "GND" (at 185.1152 87.884) (layer "F.SilkS")
+    (effects (font (size 1.5 1.5) (thickness 0.3)))
+  )
+  (gr_text "GND Green" (at 288.9504 71.628) (layer "F.SilkS")
+    (effects (font (size 1.5 1.5) (thickness 0.3)))
+  )
+  (gr_text "GND" (at 162.052 7.4168) (layer "F.SilkS")
+    (effects (font (size 1.5 1.5) (thickness 0.3)))
+  )
+  (gr_text "GND" (at 287.3756 58.166) (layer "F.SilkS")
+    (effects (font (size 1.5 1.5) (thickness 0.3)))
+  )
+  (gr_text "12VDC out" (at 289.0012 82.0928) (layer "F.SilkS")
+    (effects (font (size 1.5 1.5) (thickness 0.3)))
+  )
+  (gr_text "GND" (at 265.2268 87.9856) (layer "F.SilkS")
+    (effects (font (size 1.5 1.5) (thickness 0.3)))
+  )
   (gr_text "Analog LED Strip Controller V0.1\nRandall Shutt\nrandall@randallman.net" (at 220.8276 6.4008) (layer "F.SilkS")
     (effects (font (size 1.5 1.5) (thickness 0.3)))
   )
+  (gr_text "12VDC" (at 185.8264 7.366) (layer "F.SilkS")
+    (effects (font (size 1.5 1.5) (thickness 0.3)))
+  )
+  (gr_text "GND Blue" (at 288.1884 66.7004) (layer "F.SilkS")
+    (effects (font (size 1.5 1.5) (thickness 0.3)))
+  )
+  (gr_text "GND Red" (at 287.9852 76.9112) (layer "F.SilkS")
+    (effects (font (size 1.5 1.5) (thickness 0.3)))
+  )
+  (gr_text "+12VDC" (at 287.6804 52.6796) (layer "F.SilkS")
+    (effects (font (size 1.5 1.5) (thickness 0.3)))
+  )
+  (gr_text "12VDC" (at 161.6964 87.7824) (layer "F.SilkS")
+    (effects (font (size 1.5 1.5) (thickness 0.3)))
+  )
+  (gr_text "12VDC" (at 280.5684 7.7724) (layer "F.SilkS")
+    (effects (font (size 1.5 1.5) (thickness 0.3)))
+  )
+  (gr_text "GND" (at 255.4732 7.7216) (layer "F.SilkS")
+    (effects (font (size 1.5 1.5) (thickness 0.3)))
+  )
+  (gr_text "12VDC" (at 241.6048 87.7824) (layer "F.SilkS")
+    (effects (font (size 1.5 1.5) (thickness 0.3)))
+  )
