File: lm224-3lows-1hi.kicad_pcb (KiCad board)
At the start: 2 copper layers, 144.6 x 105.9 mm, 38 parts, among them J1 Power, J2 To LEDs, Q1 IRLB8721, Q2 IRLB8721, Q3 IRF5210L, Q4 IRLB8721, Q5 IRLB8721, U1 LM224

Commit message: Ok more stuff
Parts:
- RV1: value 10k -> To 10k Pot - Master Brightness
- RV2: value 10k -> To 10k Pot - Red
- RV3: value 10k -> To 10k Pot - Blue
- RV4: value 10k -> To 10k Pot - Green
Other:
- board text added: "+12VDC"
- board text added: "12VDC"
- board text added: "12VDC out"
- board text added: "GND"
- board text added: "GND Blue"
- board text added: "GND Green"
- board text added: "GND Red"
Changed lines of the file:
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@@
       (outputformat 1)
       (mirror false)
-      (drillshape 1)
+      (drillshape 0)
       (scaleselection 1)
       (outputdirectory "")
@@
     (property "Sheetname" "")
     (attr through_hole)
-    (fp_text reference "J1" (at 2.54 -6.26 90) (layer "F.SilkS")
-      (effects (font (size 1 1) (thickness 0.15)))
-    )
-    (fp_text value "Power" (at 2.54 5.66 90) (layer "F.Fab")
+    (fp_text reference "J1" (at 2.6212 -7.163) (layer "F.SilkS")
+      (effects (font (size 1 1) (thickness 0.15)))
+    )
+    (fp_text value "Power" (at 9.022 -0.559) (layer "F.Fab")
       (effects (font (size 1 1) (thickness 0.15)))
     )
@@
       (effects (font (size 1 1) (thickness 0.15)))
     )
-    (fp_text value "10k" (at 5.08 5.66) (layer "F.Fab")
+    (fp_text value "To 10k Pot - Red" (at 4.8818 6.1466) (layer "F.SilkS")
       (effects (font (size 1 1) (thickness 0.15)))
     )
@@
       (effects (font (size 1 1) (thickness 0.15)))
     )
-    (fp_text value "10k" (at 5.08 5.66) (layer "F.Fab")
+    (fp_text value "To 10k Pot - Master Brightness" (at 5.1308 6.2992) (layer "F.SilkS")
       (effects (font (size 1 1) (thickness 0.15)))
     )
@@
     (property "Sheetname" "")
     (attr through_hole)
-    (fp_text reference "J2" (at 7.62 -6.26 90) (layer "F.SilkS")
-      (effects (font (size 1 1) (thickness 0.15)))
-    )
-    (fp_text value "To LEDs" (at 7.62 5.66 90) (layer "F.Fab")
+    (fp_text reference "J2" (at 19.7612 -0.2796 180) (layer "F.SilkS")
+      (effects (font (size 1 1) (thickness 0.15)))
+    )
+    (fp_text value "To LEDs" (at -4.4704 -0.0764 180) (layer "F.Fab")
       (effects (font (size 1 1) (thickness 0.15)))
     )
@@
       (effects (font (size 1 1) (thickness 0.15)))
     )
-    (fp_text value "10k" (at 5.08 5.66) (layer "F.Fab")
+    (fp_text value "To 10k Pot - Blue" (at 5.1358 6.1974) (layer "F.SilkS")
       (effects (font (size 1 1) (thickness 0.15)))
     )
@@
     (property "Sheetname" "")
     (attr through_hole)
-    (fp_text reference "U1" (at 3.81 -2.33 90) (layer "F.SilkS")
+    (fp_text reference "U1" (at 10.8612 7.5488 180) (layer "F.SilkS")
       (effects (font (size 1 1) (thickness 0.15)))
     )
@@
       (effects (font (size 1 1) (thickness 0.15)))
     )
-    (fp_text value "10k" (at 5.08 5.66) (layer "F.Fab")
+    (fp_text value "To 10k Pot - Green" (at 5.08 6.2482) (layer "F.SilkS")
       (effects (font (size 1 1) (thickness 0.15)))
     )
@@
   )
   (gr_rect (start 297.1292 0) (end 152.5016 105.8672) (layer "Edge.Cuts") (width 0.1) (fill none))
+  (gr_text "GND" (at 185.1152 87.884) (layer "F.SilkS")
+    (effects (font (size 1.5 1.5) (thickness 0.3)))
+  )
+  (gr_text "GND Green" (at 288.9504 71.628) (layer "F.SilkS")
+    (effects (font (size 1.5 1.5) (thickness 0.3)))
+  )
+  (gr_text "GND" (at 162.052 7.4168) (layer "F.SilkS")
+    (effects (font (size 1.5 1.5) (thickness 0.3)))
+  )
+  (gr_text "GND" (at 287.3756 58.166) (layer "F.SilkS")
+    (effects (font (size 1.5 1.5) (thickness 0.3)))
+  )
+  (gr_text "12VDC out" (at 289.0012 82.0928) (layer "F.SilkS")
+    (effects (font (size 1.5 1.5) (thickness 0.3)))
+  )
+  (gr_text "GND" (at 265.2268 87.9856) (layer "F.SilkS")
+    (effects (font (size 1.5 1.5) (thickness 0.3)))
+  )
   (gr_text "Analog LED Strip Controller V0.1\nRandall Shutt\nrandall@randallman.net" (at 220.8276 6.4008) (layer "F.SilkS")
     (effects (font (size 1.5 1.5) (thickness 0.3)))
   )
+  (gr_text "12VDC" (at 185.8264 7.366) (layer "F.SilkS")
+    (effects (font (size 1.5 1.5) (thickness 0.3)))
+  )
+  (gr_text "GND Blue" (at 288.1884 66.7004) (layer "F.SilkS")
+    (effects (font (size 1.5 1.5) (thickness 0.3)))
+  )
+  (gr_text "GND Red" (at 287.9852 76.9112) (layer "F.SilkS")
+    (effects (font (size 1.5 1.5) (thickness 0.3)))
+  )
+  (gr_text "+12VDC" (at 287.6804 52.6796) (layer "F.SilkS")
+    (effects (font (size 1.5 1.5) (thickness 0.3)))
+  )
+  (gr_text "12VDC" (at 161.6964 87.7824) (layer "F.SilkS")
+    (effects (font (size 1.5 1.5) (thickness 0.3)))
+  )
+  (gr_text "12VDC" (at 280.5684 7.7724) (layer "F.SilkS")
+    (effects (font (size 1.5 1.5) (thickness 0.3)))
+  )
+  (gr_text "GND" (at 255.4732 7.7216) (layer "F.SilkS")
+    (effects (font (size 1.5 1.5) (thickness 0.3)))
+  )
+  (gr_text "12VDC" (at 241.6048 87.7824) (layer "F.SilkS")
+    (effects (font (size 1.5 1.5) (thickness 0.3)))
+  )

Commit message: Ok this is another checkpoint
Parts:
- moved H3 66.7 mm to (251.3, 54.0)
- moved Q3 64.9 mm to (222.3, 89.7)
- moved R1 64.9 mm to (227.7, 70.0)
- moved R2 64.9 mm to (122.1, 70.0)
- moved RV1 64.9 mm to (232.8, 58.8)
- moved C1 64.9 mm to (190.8, 70.1)
- moved C2 64.9 mm to (168.3, 70.1)
- moved C3 64.9 mm to (164.8, 127.1)
- moved C4 64.9 mm to (184.8, 117.0)
- moved J1 64.9 mm to (237.2, 108.7)
- moved Q1 64.9 mm to (198.5, 79.6)
- moved Q2 64.9 mm to (173.0, 79.6)
- moved Q4 64.9 mm to (166.3, 118.3)
- moved Q5 64.9 mm to (180.9, 127.8)
- moved R10 64.9 mm to (196.0, 89.7)
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Routing:
- net Net-(C1-Pad1): track 66.3 -> 65.1 mm
Other:
- board size 144.6 x 105.9 mm -> 136.3 x 101.5 mm
- board text added: "12V"
- board text added: "Blue"
- board text added: "Green"
- board text added: "Red"
- board text removed: "12VDC out"
- board text removed: "GND Blue"
- board text removed: "GND Green"
- board text removed: "GND Red"
